File: HW/KiCAD/ega-right-kb.kicad_sch (KiCad schematic)
At the start: 101 parts, among them SW1 SW_Push, SW10 SW_Push, SW11 SW_Push, SW12 SW_Push, SW13 SW_Push, SW14 SW_Push, SW15 SW_Push, SW16 SW_Push, SW17 SW_Push, SW18 SW_Push, SW19 SW_Push, SW2 SW_Push, SW20 SW_Push, SW21 SW_Push, SW22 SW_Push, SW23 SW_Push, SW24 SW_Push, SW25 SW_Push, SW26 SW_Push, SW27 SW_Push, SW28 SW_Push, SW29 SW_Push, SW3 SW_Push, SW30 SW_Push, SW31 SW_Push, SW32 SW_Push, SW33 SW_Push, SW34 SW_Push, SW35 SW_Push, SW36 SW_Push, SW37 SW_Push, SW38 SW_Push, SW39 SW_Push, SW4 SW_Push, SW40 SW_Push, SW41 SW_Push, SW42 SW_Push, SW43 SW_Push, SW44 SW_Push, SW45 SW_Push, SW46 SW_Push, SW47 SW_Push, SW48 SW_Push, SW49 SW_Push, SW5 SW_Push, SW50 SW_Push, SW6 SW_Push, SW7 SW_Push, SW8 SW_Push, SW9 SW_Push

Commit message: feat: 回路図修正
Parts:
- added D29, D38, D48, D49, D56, D57: D, Diode_THT:D_DO-35_SOD27_P7.62mm_Horizontal, symbol Device:D
- added SW29, SW38, SW48, SW49, SW56, SW57: SW_Push, KeySwitch:MX-Hotswap-1U, symbol Switch:SW_Push
- renumbered D1 to D00, D2 to D01, D3 to D02, D4 to D03, D5 to D04, D6 to D05, D7 to D06, D8 to D07, D9 to D08, D29 to D30, D30 to D31, D31 to D32, D32 to D33, D33 to D34, D34 to D35, D35 to D36, D36 to D37, D37 to D40, D38 to D41, D39 to D42, D40 to D43, D41 to D44, D42 to D45, D43 to D46, D44 to D47, D45 to D50, D46 to D51, D47 to D52, D48 to D53, D49 to D54, D50 to D55, SW1 to SW00, SW2 to SW01, SW3 to SW02, SW4 to SW03, SW5 to SW04, SW6 to SW05, SW7 to SW06, SW8 to SW07, SW9 to SW08, SW29 to SW30, SW30 to SW31, SW31 to SW32, SW32 to SW33, SW33 to SW34, SW34 to SW35, SW35 to SW36, SW36 to SW37, SW37 to SW40, SW38 to SW41, SW39 to SW42, SW40 to SW43, SW41 to SW44, SW42 to SW45, SW43 to SW46, SW44 to SW47, SW45 to SW50, SW46 to SW51, SW47 to SW52, SW48 to SW53, SW49 to SW54, SW50 to SW55
Connections:
- net Col6: now also SW56.1
- net Col7: now also SW57.1
- net Col8: now also SW38.1, SW48.1
- net Col9: now also SW29.1, SW49.1
- net Row0: now also D00.2 (A), D01.2 (A), D02.2 (A), D03.2 (A), D04.2 (A), D05.2 (A), D06.2 (A), D07.2 (A), D08.2 (A); no longer D00.1 (K), D01.1 (K), D02.1 (K), D03.1 (K), D04.1 (K), D05.1 (K), D06.1 (K), D07.1 (K), D08.1 (K)
- net Row1: now also D10.2 (A), D11.2 (A), D12.2 (A), D13.2 (A), D14.2 (A), D15.2 (A), D16.2 (A), D17.2 (A), D18.2 (A), D19.2 (A); no longer D10.1 (K), D11.1 (K), D12.1 (K), D13.1 (K), D14.1 (K), D15.1 (K), D16.1 (K), D17.1 (K), D18.1 (K), D19.1 (K)
- net Row2: now also D20.2 (A), D21.2 (A), D22.2 (A), D23.2 (A), D24.2 (A), D25.2 (A), D26.2 (A), D27.2 (A), D28.2 (A), D29.2 (A); no longer D20.1 (K), D21.1 (K), D22.1 (K), D23.1 (K), D24.1 (K), D25.1 (K), D26.1 (K), D27.1 (K), D28.1 (K)
- net Row3: now also D30.2 (A), D31.2 (A), D32.2 (A), D33.2 (A), D34.2 (A), D35.2 (A), D36.2 (A), D37.2 (A), D38.2 (A); no longer D30.1 (K), D31.1 (K), D32.1 (K), D33.1 (K), D34.1 (K), D35.1 (K), D36.1 (K), D37.1 (K)
- net Row4: now also D40.2 (A), D41.2 (A), D42.2 (A), D43.2 (A), D44.2 (A), D45.2 (A), D46.2 (A), D47.2 (A), D48.2 (A), D49.2 (A); no longer D40.1 (K), D41.1 (K), D42.1 (K), D43.1 (K), D44.1 (K), D45.1 (K), D46.1 (K), D47.1 (K)
- net Row5: now also D50.2 (A), D51.2 (A), D52.2 (A), D53.2 (A), D54.2 (A), D55.2 (A), D56.2 (A), D57.2 (A); no longer D50.1 (K), D51.1 (K), D52.1 (K), D53.1 (K), D54.1 (K), D55.1 (K)
- net at SW54.2: now also D54.1 (K); no longer D54.2 (A)
- net at SW02.2: now also D02.1 (K); no longer D02.2 (A)
- net at SW41.2: now also D41.1 (K); no longer D41.2 (A)
- net at SW07.2: now also D07.1 (K); no longer D07.2 (A)
- net at SW40.2: now also D40.1 (K); no longer D40.2 (A)
- net at SW04.2: now also D04.1 (K); no longer D04.2 (A)
- net at SW33.2: now also D33.1 (K); no longer D33.2 (A)
- net at SW44.2: now also D44.1 (K); no longer D44.2 (A)
- net at SW10.2: now also D10.1 (K); no longer D10.2 (A)
- net at SW31.2: now also D31.1 (K); no longer D31.2 (A)
- net at SW25.2: now also D25.1 (K); no longer D25.2 (A)
- net at SW43.2: now also D43.1 (K); no longer D43.2 (A)
- net at SW46.2: now also D46.1 (K); no longer D46.2 (A)
- net at SW06.2: now also D06.1 (K); no longer D06.2 (A)
- net at SW15.2: now also D15.1 (K); no longer D15.2 (A)
- net at SW19.2: now also D19.1 (K); no longer D19.2 (A)
- net at SW17.2: now also D17.1 (K); no longer D17.2 (A)
- net at SW32.2: now also D32.1 (K); no longer D32.2 (A)
- net at SW45.2: now also D45.1 (K); no longer D45.2 (A)
- net at SW37.2: now also D37.1 (K); no longer D37.2 (A)
- net at SW21.2: now also D21.1 (K); no longer D21.2 (A)
- net at SW55.2: now also D55.1 (K); no longer D55.2 (A)
- net at SW35.2: now also D35.1 (K); no longer D35.2 (A)
- net at SW22.2: now also D22.1 (K); no longer D22.2 (A)
- net at SW24.2: now also D24.1 (K); no longer D24.2 (A)
- net at SW53.2: now also D53.1 (K); no longer D53.2 (A)
- net at SW27.2: now also D27.1 (K); no longer D27.2 (A)
- net at SW51.2: now also D51.1 (K); no longer D51.2 (A)
- net at SW36.2: now also D36.1 (K); no longer D36.2 (A)
- net at SW11.2: now also D11.1 (K); no longer D11.2 (A)
- net at SW34.2: now also D34.1 (K); no longer D34.2 (A)
- net at SW47.2: now also D47.1 (K); no longer D47.2 (A)
- net at SW05.2: now also D05.1 (K); no longer D05.2 (A)
- net at SW16.2: now also D16.1 (K); no longer D16.2 (A)
- net at SW20.2: now also D20.1 (K); no longer D20.2 (A)
- net at SW00.2: now also D00.1 (K); no longer D00.2 (A)
- net at SW12.2: now also D12.1 (K); no longer D12.2 (A)
- net at SW23.2: now also D23.1 (K); no longer D23.2 (A)
- net at SW01.2: now also D01.1 (K); no longer D01.2 (A)
- net at SW14.2: now also D14.1 (K); no longer D14.2 (A)
- net at SW18.2: now also D18.1 (K); no longer D18.2 (A)
- net at SW30.2: now also D30.1 (K); no longer D30.2 (A)
- net at SW42.2: now also D42.1 (K); no longer D42.2 (A)
- net at SW52.2: now also D52.1 (K); no longer D52.2 (A)
- net at SW50.2: now also D50.1 (K); no longer D50.2 (A)
- net at SW26.2: now also D26.1 (K); no longer D26.2 (A)
- net at SW03.2: now also D03.1 (K); no longer D03.2 (A)
- net at SW28.2: now also D28.1 (K); no longer D28.2 (A)
- net at SW08.2: now also D08.1 (K); no longer D08.2 (A)
- net at SW13.2: now also D13.1 (K); no longer D13.2 (A)
- new net: D56.1 (K), SW56.2
- new net: D48.1 (K), SW48.2
- new net: D38.1 (K), SW38.2
- new net: D29.1 (K), SW29.2
- new net: D57.1 (K), SW57.2
- new net: D49.1 (K), SW49.2
Other:
- moved on the sheet: D37, D47

Commit message: chore: update code structure for improved readability and maintainability
Parts:
- SW00, SW01, SW02, SW03, SW04, SW05, SW06, SW07, SW08, SW10, SW11, SW12, SW13, SW14, SW15, SW16, SW17, SW18, SW19, SW20, SW21, SW22, SW23, SW24, SW25, SW26, SW27, SW28, SW29, SW30, SW31, SW32, SW33, SW34, SW35, SW36, SW37, SW38, SW40, SW41, SW42, SW43, SW44, SW45, SW46, SW47, SW48, SW49, SW50, SW51, SW52, SW53, SW54, SW55, SW56, SW57: footprint KeySwitch:MX-Hotswap-1U -> PCM_Switch_Keyboard_Hotswap_Kailh:SW_Hotswap_Kailh_MX_1.00u

Commit message: chore: メイン基板　の配線まで完成
Parts:
- D00, D01, D02, D03, D04, D05, D06, D07, D08, D10, D11, D12, D13, D14, D15, D16, D17, D18, D19, D20, D21, D22, D23, D24, D25, D26, D27, D28, D29, D30, D31, D32, D33, D34, D35, D36, D37, D38, D40, D41, D42, D43, D44, D45, D46, D47, D48, D49, D50, D51, D52, D53, D54, D55, D56, D57: footprint Diode_THT:D_DO-35_SOD27_P7.62mm_Horizontal -> Diode_SMD:D_SOD-123
Connections:
- net Col0: now also A2.9 (GPIO6); no longer A2.6 (GPIO4)
- net Col1: now also A2.10 (GPIO7); no longer A2.7 (GPIO5)
- net Col2: now also A2.11 (GPIO8); no longer A2.9 (GPIO6)
- net Col3: now also A2.12 (GPIO9); no longer A2.10 (GPIO7)
- net Col4: now also A2.14 (GPIO10); no longer A2.11 (GPIO8)
- net Col5: now also A2.15 (GPIO11); no longer A2.12 (GPIO9)
- net Col6: now also A2.16 (GPIO12); no longer A2.5 (GPIO3)
- net Col7: now also A2.17 (GPIO13); no longer A2.4 (GPIO2)
- net Col8: now also A2.19 (GPIO14); no longer A2.2 (GPIO1)
- net Col9: now also A2.20 (GPIO15); no longer A2.1 (GPIO0)
- net Row0: now also A2.7 (GPIO5); no longer A2.27 (GPIO21)
- net Row1: now also A2.6 (GPIO4); no longer A2.26 (GPIO20)
- net Row2: now also A2.5 (GPIO3); no longer A2.25 (GPIO19)
- net Row3: now also A2.4 (GPIO2); no longer A2.24 (GPIO18)
- net Row4: now also A2.2 (GPIO1); no longer A2.22 (GPIO17)
- net Row5: now also A2.1 (GPIO0); no longer A2.21 (GPIO16)
