File: HW/KiCAD/ega-right-kb.kicad_pcb (KiCad board)
At the start: 2 copper layers, 198.1 x 154.9 mm, 101 parts, among them SW1 SW_Push, SW10 SW_Push, SW11 SW_Push, SW12 SW_Push, SW13 SW_Push, SW14 SW_Push, SW15 SW_Push, SW16 SW_Push, SW17 SW_Push, SW18 SW_Push, SW19 SW_Push, SW2 SW_Push, SW20 SW_Push, SW21 SW_Push, SW22 SW_Push, SW23 SW_Push, SW24 SW_Push, SW25 SW_Push, SW26 SW_Push, SW27 SW_Push, SW28 SW_Push, SW29 SW_Push, SW3 SW_Push, SW30 SW_Push, SW31 SW_Push, SW32 SW_Push, SW33 SW_Push, SW34 SW_Push, SW35 SW_Push, SW36 SW_Push, SW37 SW_Push, SW38 SW_Push, SW39 SW_Push, SW4 SW_Push, SW40 SW_Push, SW41 SW_Push, SW42 SW_Push, SW43 SW_Push, SW44 SW_Push, SW45 SW_Push, SW46 SW_Push, SW47 SW_Push, SW48 SW_Push, SW49 SW_Push, SW5 SW_Push, SW50 SW_Push, SW6 SW_Push, SW7 SW_Push, SW8 SW_Push, SW9 SW_Push

Commit message: chore: メイン基板　の配線まで完成
Parts:
- removed D1, D2, D3, D39, D4, D5, D6, D7, D8, D9: D, Diode_THT:D_DO-35_SOD27_P7.62mm_Horizontal
- removed SW1, SW2, SW3, SW39, SW4, SW5, SW6, SW7, SW8, SW9: SW_Push, KeySwitch:MX-Hotswap-1U
- added D00: D, Diode_SMD:D_SOD-123, B.Cu at (154.8, 68.0)
- added D01: D, Diode_SMD:D_SOD-123, B.Cu at (183.3, 68.0)
- added D02: D, Diode_SMD:D_SOD-123, B.Cu at (202.4, 68.0)
- added D03: D, Diode_SMD:D_SOD-123, B.Cu at (221.4, 68.0)
- added D04: D, Diode_SMD:D_SOD-123, B.Cu at (240.5, 68.0)
- added D05: D, Diode_SMD:D_SOD-123, B.Cu at (269.1, 68.0)
- added D06: D, Diode_SMD:D_SOD-123, B.Cu at (288.1, 68.0)
- added D07: D, Diode_SMD:D_SOD-123, B.Cu at (307.2, 68.0)
- added D08: D, Diode_SMD:D_SOD-123, B.Cu at (326.2, 68.0)
- added D51: D, Diode_SMD:D_SOD-123, B.Cu at (219.1, 172.8)
- added D52: D, Diode_SMD:D_SOD-123, B.Cu at (250.0, 172.8)
- added D53: D, Diode_SMD:D_SOD-123, B.Cu at (276.2, 172.8)
- added D54: D, Diode_SMD:D_SOD-123, B.Cu at (297.6, 172.8)
- added D55: D, Diode_SMD:D_SOD-123, B.Cu at (321.5, 177.6)
- added D56: D, Diode_SMD:D_SOD-123, B.Cu at (340.5, 177.6)
- added D57: D, Diode_SMD:D_SOD-123, B.Cu at (359.6, 177.6)
- added SW00: SW_Push, PCM_Switch_Keyboard_Hotswap_Kailh:SW_Hotswap_Kailh_MX_1.00u, F.Cu at (154.8, 59.5)
- added SW01: SW_Push, PCM_Switch_Keyboard_Hotswap_Kailh:SW_Hotswap_Kailh_MX_1.00u, F.Cu at (183.3, 59.5)
- added SW02: SW_Push, PCM_Switch_Keyboard_Hotswap_Kailh:SW_Hotswap_Kailh_MX_1.00u, F.Cu at (202.4, 59.5)
- added SW03: SW_Push, PCM_Switch_Keyboard_Hotswap_Kailh:SW_Hotswap_Kailh_MX_1.00u, F.Cu at (221.4, 59.5)
- added SW04: SW_Push, PCM_Switch_Keyboard_Hotswap_Kailh:SW_Hotswap_Kailh_MX_1.00u, F.Cu at (240.5, 59.5)
- added SW05: SW_Push, PCM_Switch_Keyboard_Hotswap_Kailh:SW_Hotswap_Kailh_MX_1.00u, F.Cu at (269.1, 59.5)
- added SW06: SW_Push, PCM_Switch_Keyboard_Hotswap_Kailh:SW_Hotswap_Kailh_MX_1.00u, F.Cu at (288.1, 59.5)
- added SW07: SW_Push, PCM_Switch_Keyboard_Hotswap_Kailh:SW_Hotswap_Kailh_MX_1.00u, F.Cu at (307.2, 59.5)
- added SW08: SW_Push, PCM_Switch_Keyboard_Hotswap_Kailh:SW_Hotswap_Kailh_MX_1.00u, F.Cu at (326.2, 59.5)
- added SW51: SW_Push, PCM_Switch_Keyboard_Hotswap_Kailh:SW_Hotswap_Kailh_MX_1.00u, F.Cu at (219.1, 164.3)
- added SW52: SW_Push, PCM_Switch_Keyboard_Hotswap_Kailh:SW_Hotswap_Kailh_MX_1.00u, F.Cu at (250.0, 164.3)
- added SW53: SW_Push, PCM_Switch_Keyboard_Hotswap_Kailh:SW_Hotswap_Kailh_MX_1.00u, F.Cu at (276.2, 164.3)
- added SW54: SW_Push, PCM_Switch_Keyboard_Hotswap_Kailh:SW_Hotswap_Kailh_MX_1.00u, F.Cu at (297.6, 164.3)
- added SW55: SW_Push, PCM_Switch_Keyboard_Hotswap_Kailh:SW_Hotswap_Kailh_MX_1.00u, F.Cu at (321.5, 169.1)
- added SW56: SW_Push, PCM_Switch_Keyboard_Hotswap_Kailh:SW_Hotswap_Kailh_MX_1.00u, F.Cu at (340.5, 169.1)
- added SW57: SW_Push, PCM_Switch_Keyboard_Hotswap_Kailh:SW_Hotswap_Kailh_MX_1.00u, F.Cu at (359.6, 169.1)
- D10, D11, D12, D13, D14, D15, D16, D17, D18, D19, D20, D21, D22, D23, D24, D25, D26, D27, D28, D29, D30, D31, D32, D33, D34, D35, D36, D37, D38, D40, D41, D42, D43, D44, D45, D46, D47, D48, D49, D50: footprint Diode_THT:D_DO-35_SOD27_P7.62mm_Horizontal -> Diode_SMD:D_SOD-123
- SW10, SW11, SW12, SW13, SW14, SW15, SW16, SW17, SW18, SW19, SW20, SW21, SW22, SW23, SW24, SW25, SW26, SW27, SW28, SW29, SW30, SW31, SW32, SW33, SW34, SW35, SW36, SW37, SW38, SW40, SW41, SW42, SW43, SW44, SW45, SW46, SW47, SW48, SW49, SW50: footprint KeySwitch:MX-Hotswap-1U -> PCM_Switch_Keyboard_Hotswap_Kailh:SW_Hotswap_Kailh_MX_1.00u; moved to F.Cu
- moved D29 300.2 mm to (350.0, 115.7), turned to 180 degrees
- moved SW29 296.2 mm to (350.0, 107.2), turned to 0 degrees
- moved D38 271.7 mm to (350.0, 134.7), turned to 180 degrees
- moved SW38 267.7 mm to (350.0, 126.2), turned to 0 degrees
- moved D37 243.2 mm to (302.4, 134.7), turned to 180 degrees
- moved SW37 239.2 mm to (302.4, 126.2), turned to 0 degrees
- moved D45 209.9 mm to (273.8, 153.8), turned to 180 degrees
- moved SW45 206.0 mm to (273.8, 145.2), turned to 0 degrees
- moved D46 193.3 mm to (292.9, 153.8), turned to 180 degrees
- moved D47 190.6 mm to (321.5, 158.5), turned to 180 degrees
- moved SW46 189.4 mm to (292.9, 145.2), turned to 0 degrees
- moved SW47 186.6 mm to (321.5, 150.0), turned to 0 degrees
- moved D48 183.4 mm to (340.5, 158.5), turned to 180 degrees
- moved SW48 179.5 mm to (340.5, 150.0), turned to 0 degrees
- moved D49 178.7 mm to (359.6, 158.5), turned to 180 degrees
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Connections:
- net Net-(A2-GND-Pad13) renamed GND
- A2 pad 1: Col9 -> Row5
- A2 pad 10: Col3 -> Col1
- A2 pad 11: Col4 -> Col2
- A2 pad 12: Col5 -> Col3
- A2 pad 14: unconnected-(A2-GPIO10-Pad14) -> Col4
- A2 pad 15: unconnected-(A2-GPIO11-Pad15) -> Col5
- A2 pad 16: unconnected-(A2-GPIO12-Pad16) -> Col6
- A2 pad 17: unconnected-(A2-GPIO13-Pad17) -> Col7
- A2 pad 19: unconnected-(A2-GPIO14-Pad19) -> Col8
- A2 pad 2: Col8 -> Row4
- A2 pad 20: unconnected-(A2-GPIO15-Pad20) -> Col9
- A2 pad 21: Row5 -> unconnected-(A2-GPIO16-Pad21)
- A2 pad 22: Row4 -> unconnected-(A2-GPIO17-Pad22)
- A2 pad 24: Row3 -> unconnected-(A2-GPIO18-Pad24)
- A2 pad 25: Row2 -> unconnected-(A2-GPIO19-Pad25)
- A2 pad 26: Row1 -> unconnected-(A2-GPIO20-Pad26)
- A2 pad 27: Row0 -> unconnected-(A2-GPIO21-Pad27)
- A2 pad 4: Col7 -> Row3
- A2 pad 5: Col6 -> Row2
- A2 pad 6: Col0 -> Row1
- A2 pad 7: Col1 -> Row0
- A2 pad 9: Col2 -> Col0
- D10 pad 1: Row1 -> Net-(D10-K)
- D10 pad 2: Net-(D10-A) -> Row1
- D11 pad 1: Row1 -> Net-(D11-K)
- D11 pad 2: Net-(D11-A) -> Row1
- D12 pad 1: Row1 -> Net-(D12-K)
- D12 pad 2: Net-(D12-A) -> Row1
- D13 pad 1: Row1 -> Net-(D13-K)
- D13 pad 2: Net-(D13-A) -> Row1
- D14 pad 1: Row1 -> Net-(D14-K)
- D14 pad 2: Net-(D14-A) -> Row1
- D15 pad 1: Row1 -> Net-(D15-K)
- D15 pad 2: Net-(D15-A) -> Row1
- D16 pad 1: Row1 -> Net-(D16-K)
- D16 pad 2: Net-(D16-A) -> Row1
- D17 pad 1: Row1 -> Net-(D17-K)
- D17 pad 2: Net-(D17-A) -> Row1
- D18 pad 1: Row1 -> Net-(D18-K)
- D18 pad 2: Net-(D18-A) -> Row1
- D19 pad 1: Row1 -> Net-(D19-K)
- D19 pad 2: Net-(D19-A) -> Row1
- D20 pad 1: Row2 -> Net-(D20-K)
- D20 pad 2: Net-(D20-A) -> Row2
- D21 pad 1: Row2 -> Net-(D21-K)
- D21 pad 2: Net-(D21-A) -> Row2
- D22 pad 1: Row2 -> Net-(D22-K)
- D22 pad 2: Net-(D22-A) -> Row2
- D23 pad 1: Row2 -> Net-(D23-K)
- D23 pad 2: Net-(D23-A) -> Row2
- D24 pad 1: Row2 -> Net-(D24-K)
- D24 pad 2: Net-(D24-A) -> Row2
- D25 pad 1: Row2 -> Net-(D25-K)
- D25 pad 2: Net-(D25-A) -> Row2
- D26 pad 1: Row2 -> Net-(D26-K)
- D26 pad 2: Net-(D26-A) -> Row2
- D27 pad 1: Row2 -> Net-(D27-K)
- D27 pad 2: Net-(D27-A) -> Row2
- D28 pad 1: Row2 -> Net-(D28-K)
- D28 pad 2: Net-(D28-A) -> Row2
- D29 pad 1: Row3 -> Net-(D29-K)
- D29 pad 2: Net-(D29-A) -> Row2
- D30 pad 1: Row3 -> Net-(D30-K)
- D30 pad 2: Net-(D30-A) -> Row3
- D31 pad 1: Row3 -> Net-(D31-K)
- D31 pad 2: Net-(D31-A) -> Row3
- D32 pad 1: Row3 -> Net-(D32-K)
- D32 pad 2: Net-(D32-A) -> Row3
- D33 pad 1: Row3 -> Net-(D33-K)
- D33 pad 2: Net-(D33-A) -> Row3
- D34 pad 1: Row3 -> Net-(D34-K)
- D34 pad 2: Net-(D34-A) -> Row3
- D35 pad 1: Row3 -> Net-(D35-K)
- D35 pad 2: Net-(D35-A) -> Row3
- D36 pad 1: Row3 -> Net-(D36-K)
- D36 pad 2: Net-(D36-A) -> Row3
- D37 pad 1: Row4 -> Net-(D37-K)
- D37 pad 2: Net-(D37-A) -> Row3
- D38 pad 1: Row4 -> Net-(D38-K)
- D38 pad 2: Net-(D38-A) -> Row3
- D40 pad 1: Row4 -> Net-(D40-K)
- D40 pad 2: Net-(D40-A) -> Row4
- D41 pad 1: Row4 -> Net-(D41-K)
- D41 pad 2: Net-(D41-A) -> Row4
- D42 pad 1: Row4 -> Net-(D42-K)
- D42 pad 2: Net-(D42-A) -> Row4
- D43 pad 1: Row4 -> Net-(D43-K)
- D43 pad 2: Net-(D43-A) -> Row4
- D44 pad 1: Row4 -> Net-(D44-K)
- D44 pad 2: Net-(D44-A) -> Row4
- D45 pad 1: Row5 -> Net-(D45-K)
- D45 pad 2: Net-(D45-A) -> Row4
- D46 pad 1: Row5 -> Net-(D46-K)
- D46 pad 2: Net-(D46-A) -> Row4
- D47 pad 1: Row5 -> Net-(D47-K)
- D47 pad 2: Net-(D47-A) -> Row4
- D48 pad 1: Row5 -> Net-(D48-K)
- D48 pad 2: Net-(D48-A) -> Row4
- D49 pad 1: Row5 -> Net-(D49-K)
- D49 pad 2: Net-(D49-A) -> Row4
- D50 pad 1: Row5 -> Net-(D50-K)
- D50 pad 2: Net-(D50-A) -> Row5
- SW10 pad 2: Net-(D10-A) -> Net-(D10-K)
- SW11 pad 2: Net-(D11-A) -> Net-(D11-K)
- SW12 pad 2: Net-(D12-A) -> Net-(D12-K)
- SW13 pad 2: Net-(D13-A) -> Net-(D13-K)
- SW14 pad 2: Net-(D14-A) -> Net-(D14-K)
- SW15 pad 2: Net-(D15-A) -> Net-(D15-K)
- SW16 pad 2: Net-(D16-A) -> Net-(D16-K)
- SW17 pad 2: Net-(D17-A) -> Net-(D17-K)
- SW18 pad 2: Net-(D18-A) -> Net-(D18-K)
- SW19 pad 2: Net-(D19-A) -> Net-(D19-K)
- SW20 pad 2: Net-(D20-A) -> Net-(D20-K)
- SW21 pad 2: Net-(D21-A) -> Net-(D21-K)
- SW22 pad 2: Net-(D22-A) -> Net-(D22-K)
- SW23 pad 2: Net-(D23-A) -> Net-(D23-K)
- SW24 pad 2: Net-(D24-A) -> Net-(D24-K)
- SW25 pad 2: Net-(D25-A) -> Net-(D25-K)
- SW26 pad 2: Net-(D26-A) -> Net-(D26-K)
- SW27 pad 2: Net-(D27-A) -> Net-(D27-K)
- SW28 pad 2: Net-(D28-A) -> Net-(D28-K)
- SW29 pad 1: Col0 -> Col9
- SW29 pad 2: Net-(D29-A) -> Net-(D29-K)
- SW30 pad 1: Col1 -> Col0
- SW30 pad 2: Net-(D30-A) -> Net-(D30-K)
- SW31 pad 1: Col2 -> Col1
- SW31 pad 2: Net-(D31-A) -> Net-(D31-K)
- SW32 pad 1: Col3 -> Col2
- SW32 pad 2: Net-(D32-A) -> Net-(D32-K)
- SW33 pad 1: Col4 -> Col3
- SW33 pad 2: Net-(D33-A) -> Net-(D33-K)
- SW34 pad 1: Col5 -> Col4
- SW34 pad 2: Net-(D34-A) -> Net-(D34-K)
- SW35 pad 1: Col6 -> Col5
- SW35 pad 2: Net-(D35-A) -> Net-(D35-K)
- SW36 pad 1: Col7 -> Col6
- SW36 pad 2: Net-(D36-A) -> Net-(D36-K)
- SW37 pad 1: Col0 -> Col7
- SW37 pad 2: Net-(D37-A) -> Net-(D37-K)
- SW38 pad 1: Col1 -> Col8
- SW38 pad 2: Net-(D38-A) -> Net-(D38-K)
- SW40 pad 1: Col3 -> Col0
- SW40 pad 2: Net-(D40-A) -> Net-(D40-K)
- SW41 pad 1: Col4 -> Col1
- SW41 pad 2: Net-(D41-A) -> Net-(D41-K)
- SW42 pad 1: Col5 -> Col2
- SW42 pad 2: Net-(D42-A) -> Net-(D42-K)
- SW43 pad 1: Col6 -> Col3
- SW43 pad 2: Net-(D43-A) -> Net-(D43-K)
- SW44 pad 1: Col7 -> Col4
- SW44 pad 2: Net-(D44-A) -> Net-(D44-K)
- SW45 pad 1: Col0 -> Col5
- SW45 pad 2: Net-(D45-A) -> Net-(D45-K)
- SW46 pad 1: Col1 -> Col6
- SW46 pad 2: Net-(D46-A) -> Net-(D46-K)
- SW47 pad 1: Col2 -> Col7
- SW47 pad 2: Net-(D47-A) -> Net-(D47-K)
- SW48 pad 1: Col3 -> Col8
- SW48 pad 2: Net-(D48-A) -> Net-(D48-K)
- SW49 pad 1: Col4 -> Col9
- SW49 pad 2: Net-(D49-A) -> Net-(D49-K)
- SW50 pad 1: Col5 -> Col0
- SW50 pad 2: Net-(D50-A) -> Net-(D50-K)
Routing:
- net Col9: track 66.8 -> 269.6 mm, vias 0 -> 3
- net Col0: track 309.4 -> 138.1 mm, vias 0 -> 6
- net Col8: track 107.9 -> 268.0 mm, vias 0 -> 5
- net Col1: track 291.5 -> 149.5 mm, vias 0 -> 6
- net Row0: track 351.6 -> 214.2 mm
- net Row1: track 376.5 -> 241.4 mm
- net GND: track 0.00 -> 133.5 mm
- net Col7: track 152.2 -> 282.4 mm, vias 0 -> 6
- net Col6: track 165.0 -> 268.9 mm, vias 0 -> 6
- net Row2: track 390.5 -> 287.3 mm
- net Col2: track 279.1 -> 178.9 mm, vias 0 -> 6
- net Row5: track 421.1 -> 331.8 mm
- net Row3: track 383.4 -> 295.2 mm
- net Row4: track 404.8 -> 319.1 mm
- net Col3: track 264.6 -> 199.0 mm, vias 0 -> 6
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Other:
- board size 198.1 x 154.9 mm -> 235.5 x 163 mm

Commit message: feat: update KiCAD project files and add production resources
- Changed active layer from 0 to 25 and updated zone display mode from 0 to 1 in `ega-right-kb.kicad_prl`.
- Added new binary file `Keyboard.zip` to the production directory.
- Created new BOM file `Keyboard_bom.csv` with component details.
- Added designators for components in `Keyboard_designators.csv`.
- Included positions for components in `Keyboard_positions.csv`.
- Updated netlist in `netlist.ipc` with new VIA specifications.
Other:
- board size 235.5 x 163 mm -> 241.3 x 170.5 mm
Changed lines of the file:
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@@
 		(legacy_teardrops no)
 	)
-	(paper "A3")
+	(paper "A2" portrait)
 	(layers
 		(0 "F.Cu" signal)
@@
 		(allow_soldermask_bridges_in_footprints no)
 		(tenting front back)
+		(grid_origin 140.25 15)
 		(pcbplotparams
 			(layerselection 0x00000000_00000000_55555555_5755f5ff)
@@
 	)
 	(gr_arc
-		(start 375 181.5)
-		(mid 374.707107 182.207107)
-		(end 374 182.5)
+		(start 140.75 183.4875)
+		(mid 140.042893 183.194607)
+		(end 139.75 182.4875)
 		(stroke
-			(width 0.05)
+			(width 0.1)
+			(type default)
+		)
+		(layer "Edge.Cuts")
+	)
+	(gr_line
+		(start 139.75 182.4875)
+		(end 139.75 14)
+		(stroke
+			(width 0.1)
 			(type default)
 		)
@@
 	)
 	(gr_arc
-		(start 139.5 20.5)
-		(mid 139.792893 19.792893)
-		(end 140.5 19.5)
+		(start 381.0875 182.4875)
+		(mid 380.794607 183.194607)
+		(end 380.0875 183.4875)
 		(stroke
-			(width 0.05)
+			(width 0.1)
 			(type default)
 		)
 		(layer "Edge.Cuts")
 	)
+	(gr_circle
+		(center 376.0875 18)
+		(end 377.5875 18)
+		(stroke
+			(width 0.1)
+			(type default)
+		)
+		(fill no)
+		(layer "Edge.Cuts")
+	)
 	(gr_arc
-		(start 140.5 182.5)
-		(mid 139.792893 182.207107)
-		(end 139.5 181.5)
+		(start 139.75 14)
+		(mid 140.042893 13.292893)
+		(end 140.75 13)
 		(stroke
-			(width 0.05)
+			(width 0.1)
 			(type default)
 		)
@@
 	)
 	(gr_line
-		(start 140.5 19.5)
-		(end 374 19.5)
+		(start 140.75 13)
+		(end 380.0875 13)
 		(stroke
-			(width 0.05)
+			(width 0.1)
 			(type default)
 		)
 		(layer "Edge.Cuts")
 	)
-	(gr_line
-		(start 374 182.5)
-		(end 140.5 182.5)
+	(gr_arc
+		(start 380.0875 13)
+		(mid 380.794607 13.292893)
+		(end 381.0875 14)
 		(stroke
-			(width 0.05)
+			(width 0.1)
 			(type default)
 		)
@@
 	)
 	(gr_line
-		(start 139.5 181.5)
-		(end 139.5 20.5)
+		(start 380.0875 183.4875)
+		(end 140.75 183.4875)
 		(stroke
-			(width 0.05)
+			(width 0.1)
 			(type default)
 		)
 		(layer "Edge.Cuts")
 	)
-	(gr_arc
-		(start 374 19.5)
-		(mid 374.707107 19.792893)
-		(end 375 20.5)
+	(gr_circle
+		(center 144.75 178.4875)
+		(end 146.25 178.4875)
+		(stroke
+			(width 0.1)
+			(type default)
+		)
+		(fill no)
+		(layer "Edge.Cuts")
+	)
+	(gr_circle
+		(center 144.75 18)
+		(end 146.25 18)
+		(stroke
+			(width 0.1)
+			(type default)
+		)
+		(fill no)
+		(layer "Edge.Cuts")
+	)
+	(gr_circle
+		(center 376.0875 178.4875)
+		(end 377.5875 178.4875)
 		(stroke
-			(width 0.05)
+			(width 0.1)
 			(type default)
 		)
+		(fill no)
 		(layer "Edge.Cuts")
 	)
 	(gr_line
-		(start 375 20.5)
-		(end 375 181.5)
+		(start 381.0875 14)
+		(end 381.0875 182.4875)
 		(stroke
-			(width 0.05)
+			(width 0.1)
 			(type default)
 		)
